Commit message: zed URDF corrections

File: src/caramelo_bringup/urdf/caramelo_real.urdf.xacro (robot description, xacro)
@@ -43,5 +43,5 @@
     frame_id="laser_frame"
     xyz_offset="0.292 0 0.077"
-    rpy_offset="0 0 0"
+    rpy_offset="0 0 ${-M_PI}"
     mesh_xyz_offset="0 0 0"
     mesh_rpy_offset="0 0 0"

File: src/caramelo_description/URDF/robot.urdf.xacro (robot description, xacro)
@@ -44,5 +44,5 @@
     frame_id="laser_frame"
     xyz_offset="0.292 0 0.077"
-    rpy_offset="0 0 0"
+    rpy_offset="0 0 ${-M_PI}"
     mesh_xyz_offset="0 0 0"
     mesh_rpy_offset="0 0 0"

File: src/caramelo_description/URDF/zed_camera.xacro (robot description, xacro)
@@ -1,16 +1,14 @@
 <?xml version="1.0"?>
 <robot xmlns:xacro="http://www.ros.org/wiki/xacro">
-  <!-- Propriedades da ZED 2i baseadas no padrão oficial -->
-  <xacro:property name="M_PI" value="3.1415926535897931"/>
-  <xacro:property name="zed2i_baseline" value="0.12"/>    <!-- Distância entre câmeras -->
-  <xacro:property name="zed2i_height" value="0.03"/>      <!-- Altura da ZED 2i -->
-  <xacro:property name="zed2i_bottom_slope" value="0.0"/>
-  <xacro:property name="zed2i_screw_offset_x" value="-0.01"/>
-  <xacro:property name="zed2i_screw_offset_z" value="0.0"/>
-  <xacro:property name="zed2i_optical_offset_x" value="-0.01"/>
-  <!-- Dimensões físicas para visualização -->
-  <xacro:property name="zed2i_width" value="0.175"/>     <!-- Largura -->
-  <xacro:property name="zed2i_depth" value="0.030"/>     <!-- Profundidade -->
-  <xacro:property name="zed2i_mass" value="0.159"/>      <!-- Massa em kg -->
+  <!-- Propriedades da ZED 2i -->
+  <xacro:property name="zed_baseline" value="0.12"/>  <!-- Distância entre câmeras estéreo -->
+  <xacro:property name="zed_height" value="0.033"/>   <!-- Altura da ZED 2i -->
+  <xacro:property name="zed_bottom_clearance" value="0.004"/>
+  <xacro:property name="zed_screw_offset_x" value="0.0"/>
+  <xacro:property name="zed_screw_offset_z" value="0.0"/>
+  <!-- Dimensões físicas da ZED 2i -->
+  <xacro:property name="zed_width" value="0.175"/>    <!-- Largura -->
+  <xacro:property name="zed_depth" value="0.030"/>    <!-- Profundidade -->
+  <xacro:property name="zed_mass" value="0.159"/>     <!-- Massa em kg -->
   <!-- Macro da câmera ZED 2i -->
   <xacro:macro name="zed_camera" params="
@@ -26,28 +24,26 @@
     <joint name="${prefix}${frame_id}_joint" type="fixed">
       <parent link="${parent}"/>
-      <child link="${prefix}${frame_id}_camera_link"/>
+      <child link="${prefix}${frame_id}"/>
       <origin xyz="${xyz_offset}" rpy="${rpy_offset}"/>
     </joint>
-    <!-- Camera mounting point (ponto de montagem da câmera) -->
-    <link name="${prefix}${frame_id}_camera_link"/>
-    <!-- Camera Center (centro da câmera) -->
-    <link name="${prefix}${frame_id}_camera_center">
+    <!-- Link principal da ZED -->
+    <link name="${prefix}${frame_id}">
       <visual>
-        <origin xyz="${zed2i_screw_offset_x} 0 ${zed2i_screw_offset_z}" rpy="0 0 0"/>
+        <origin xyz="${mesh_xyz_offset}" rpy="${mesh_rpy_offset}"/>
         <geometry>
-          <box size="${zed2i_depth} ${zed2i_width} ${zed2i_height}"/>
+          <box size="${zed_width} ${zed_depth} ${zed_height}"/>
         </geometry>
-        <material name="zed2i_mat">
+        <material name="zed_mat">
           <color rgba="0.25 0.25 0.25 0.99"/>
         </material>
       </visual>
       <collision>
-        <origin xyz="${zed2i_screw_offset_x} 0 ${zed2i_screw_offset_z}" rpy="0 0 0"/>
+        <origin xyz="0 0 0" rpy="0 0 0"/>
         <geometry>
-          <box size="${zed2i_depth} ${zed2i_width} ${zed2i_height}"/>
+          <box size="${zed_width} ${zed_depth} ${zed_height}"/>
         </geometry>
       </collision>
       <inertial>
-        <mass value="${zed2i_mass}"/>
+        <mass value="${zed_mass}"/>
         <origin xyz="0 0 0" rpy="0 0 0"/>
         <inertia ixx="0.000239" ixy="0.0" ixz="0.0"
@@ -56,48 +52,45 @@
       </inertial>
     </link>
-    <joint name="${prefix}${frame_id}_camera_center_joint" type="fixed">
-      <parent link="${prefix}${frame_id}_camera_link"/>
-      <child link="${prefix}${frame_id}_camera_center"/>
-      <origin xyz="0 0 ${zed2i_height/2}" rpy="0 ${zed2i_bottom_slope} 0"/>
-    </joint>
-    <!-- Left Camera -->
+    <!-- Link da câmera esquerda -->
+    <joint name="${prefix}${frame_id}_left_camera_joint" type="fixed">
+      <parent link="${prefix}${frame_id}"/>
+      <child link="${prefix}${frame_id}_left_camera_frame"/>
+      <origin xyz="0 ${zed_baseline/2} 0" rpy="0 0 0"/>
+    </joint>
     <link name="${prefix}${frame_id}_left_camera_frame"/>
-    <joint name="${prefix}${frame_id}_left_camera_joint" type="fixed">
-      <parent link="${prefix}${frame_id}_camera_center"/>
-      <child link="${prefix}${frame_id}_left_camera_frame"/>
-      <origin xyz="${zed2i_optical_offset_x} ${zed2i_baseline/2} 0" rpy="0 0 0"/>
-    </joint>
-    <link name="${prefix}${frame_id}_left_camera_optical_frame"/>
+    <!-- Joint da câmera esquerda optical -->
     <joint name="${prefix}${frame_id}_left_camera_optical_joint" type="fixed">
-      <origin xyz="0 0 0" rpy="-${M_PI/2} 0.0 -${M_PI/2}"/>
       <parent link="${prefix}${frame_id}_left_camera_frame"/>
       <child link="${prefix}${frame_id}_left_camera_optical_frame"/>
-    </joint>
-    <!-- Right Camera -->
+      <origin xyz="0 0 0" rpy="-1.5708 0 -1.5708"/>
+    </joint>
+    <link name="${prefix}${frame_id}_left_camera_optical_frame"/>
+    <!-- Link da câmera direita -->
+    <joint name="${prefix}${frame_id}_right_camera_joint" type="fixed">
+      <parent link="${prefix}${frame_id}"/>
+      <child link="${prefix}${frame_id}_right_camera_frame"/>
+      <origin xyz="0 -${zed_baseline/2} 0" rpy="0 0 0"/>
+    </joint>
     <link name="${prefix}${frame_id}_right_camera_frame"/>
-    <joint name="${prefix}${frame_id}_right_camera_joint" type="fixed">
-      <parent link="${prefix}${frame_id}_camera_center"/>
-      <child link="${prefix}${frame_id}_right_camera_frame"/>
-      <origin xyz="${zed2i_optical_offset_x} -${zed2i_baseline/2} 0" rpy="0 0 0"/>
-    </joint>
-    <link name="${prefix}${frame_id}_right_camera_optical_frame"/>
+    <!-- Joint da câmera direita optical -->
     <joint name="${prefix}${frame_id}_right_camera_optical_joint" type="fixed">
-      <origin xyz="0 0 0" rpy="-${M_PI/2} 0.0 -${M_PI/2}"/>
       <parent link="${prefix}${frame_id}_right_camera_frame"/>
       <child link="${prefix}${frame_id}_right_camera_optical_frame"/>
-    </joint>
-    <!-- IMU Link (integrado na ZED 2i) -->
-    <link name="${prefix}${frame_id}_imu_link"/>
+      <origin xyz="0 0 0" rpy="-1.5708 0 -1.5708"/>
+    </joint>
+    <link name="${prefix}${frame_id}_right_camera_optical_frame"/>
+    <!-- IMU Link -->
     <joint name="${prefix}${frame_id}_imu_joint" type="fixed">
-      <parent link="${prefix}${frame_id}_camera_center"/>
+      <parent link="${prefix}${frame_id}"/>
       <child link="${prefix}${frame_id}_imu_link"/>
       <origin xyz="0 0 0" rpy="0 0 0"/>
     </joint>
+    <link name="${prefix}${frame_id}_imu_link"/>
     <!-- Plugin do Gazebo para a ZED (Ignition Gazebo) -->
     <xacro:if value="${is_ignition}">
-      <gazebo reference="${prefix}${frame_id}_camera_center">
-        <!-- Plugin da câmera estéreo esquerda -->
+      <gazebo reference="${prefix}${frame_id}">
+        <!-- Plugin da câmera estéreo -->
         <sensor name="zed_left_camera" type="camera">
-          <pose>${zed2i_optical_offset_x} ${zed2i_baseline/2} 0 0 0 0</pose>
+          <pose>0 ${zed_baseline/2} 0 0 0 0</pose>
           <camera>
             <horizontal_fov>1.919</horizontal_fov>
@@ -122,7 +115,6 @@
           <topic>zed/left/image_rect_color</topic>
         </sensor>
-        <!-- Plugin da câmera estéreo direita -->
         <sensor name="zed_right_camera" type="camera">
-          <pose>${zed2i_optical_offset_x} -${zed2i_baseline/2} 0 0 0 0</pose>
+          <pose>0 -${zed_baseline/2} 0 0 0 0</pose>
           <camera>
             <horizontal_fov>1.919</horizontal_fov>
@@ -149,5 +141,5 @@
         <!-- Plugin da câmera de profundidade -->
         <sensor name="zed_depth_camera" type="depth_camera">
-          <pose>${zed2i_optical_offset_x} 0 0 0 0 0</pose>
+          <pose>0 0 0 0 0 0</pose>
           <camera>
             <horizontal_fov>1.919</horizontal_fov>

Commit message: TF tree analizys

File: src/caramelo_bringup/urdf/caramelo_real.urdf.xacro (robot description, xacro)
@@ -47,14 +47,41 @@
     mesh_rpy_offset="0 0 0"
     topic_name="scan"/>
-  <!-- ZED 2i Camera - Posicionada no centro especificado -->
-  <xacro:zed_camera
-    prefix="$(arg prefix)"
-    parent="base_link"
-    frame_id="zed_camera"
-    xyz_offset="0.291 0 0.116"
-    rpy_offset="0 0 0"
-    mesh_xyz_offset="0 0 0"
-    mesh_rpy_offset="0 0 ${M_PI/2}"
-    is_ignition="$(arg is_ignition)"/>
+  <!-- ZED 2i Camera Link - Frame base que a ZED espera -->
+  <joint name="zed_camera_link_joint" type="fixed">
+    <parent link="base_link"/>
+    <child link="zed_camera_link"/>
+    <origin xyz="0.291 0 0.116" rpy="0 0 0"/>
+  </joint>
+  <link name="zed_camera_link">
+    <visual>
+      <origin xyz="0 0 0" rpy="0 0 ${M_PI/2}"/>
+      <geometry>
+        <box size="0.175 0.030 0.033"/>
+      </geometry>
+      <material name="zed_mat">
+        <color rgba="0.25 0.25 0.25 0.99"/>
+      </material>
+    </visual>
+    <collision>
+      <origin xyz="0 0 0" rpy="0 0 0"/>
+      <geometry>
+        <box size="0.175 0.030 0.033"/>
+      </geometry>
+    </collision>
+    <inertial>
+      <mass value="0.159"/>
+      <origin xyz="0 0 0" rpy="0 0 0"/>
+      <inertia ixx="0.000239" ixy="0.0" ixz="0.0"
+               iyy="0.000239" iyz="0.0"
+               izz="0.000451"/>
+    </inertial>
+  </link>
+  <!-- ZED 2i IMU Link - Frame da IMU que a ZED publica -->
+  <joint name="zed_imu_link_joint" type="fixed">
+    <parent link="zed_camera_link"/>
+    <child link="zed_imu_link"/>
+    <origin xyz="0 0 0" rpy="0 0 0"/>
+  </joint>
+  <link name="zed_imu_link"/>
   <!-- =============================================== -->
   <!-- ROS 2 Control Configuration for REAL HARDWARE -->
